Commit message: added files

File: eca_a9_description/urdf/eca_a9_base.xacro (robot description, xacro)
@@ -20,5 +20,5 @@
   <!-- Properties -->
   <xacro:property name="mass" value="69.7"/>
-  <xacro:property name="length" value="1.98"/>
+  <xacro:property name="length" value="19.8"/>
   <xacro:property name="diameter" value="0.23"/>
   <xacro:property name="radius" value="${diameter*0.5}"/>
@@ -37,5 +37,5 @@
         <origin xyz="0 0 0" rpy="0 0 0"/>
         <geometry>
-          <mesh filename="${visual_mesh_file}" scale="1 1 1" />
+          <mesh filename="${visual_mesh_file}" scale="40 40 40" />
         </geometry>
       </visual>
@@ -43,5 +43,5 @@
         <origin xyz="0 0 0" rpy="0 0 0"/>
         <geometry>
-          <mesh filename="${visual_mesh_file}" scale="1 1 1" />
+          <mesh filename="${visual_mesh_file}" scale="40 40 40" />
         </geometry>
       </collision>
